File: karmacontroller.brd (EAGLE design)
At the start: 100 x 50 mm, 19 parts

Commit message: v1.1 for first production PCB print
Parts:
- moved R1 9.25 mm to (31.8, 49.5)
- moved R10 7.62 mm to (16.5, 52.1)
- moved R5 7.18 mm to (55.9, 47.0), turned to 0 degrees
- moved S4 1.27 mm to (17.8, 68.6)
Routing:
- net 5V: track 281.3 -> 269.1 mm
- net DOWN: track 27.6 -> 25.0 mm
- net N$4: track 50.9 -> 53.2 mm
Other:
- outline, holes or cut-outs redrawn
- board text added: "5V"
- board text added: "GND"
- board text added: "Karma Controller v1.1 Kit 4/16/2013 William Wnekowicz w/ Zack Freedman at MakerBar"
- board text removed: "v1.0 William Wnekowicz"
